Commit message: INTERGRATE IGN TO ROS2

File: description/macros.xacro (robot description, xacro)
@@ -2,12 +2,30 @@
 <robot xmlns:xacro="http://www.ros.org/wiki/xacro">
     <!--................................ INERTIA MATRICES .............................. -->
-    <xacro:macro name="cylinder_inertia" params="m r h">
-        <inertia ixx="${m * (3 * r * r + h * h) / 12}" ixy="0" ixz="0" iyy="${m * (3 * r * r + h * h) / 12}" iyz="0" izz="${m * r * r / 2}" />
+    <xacro:macro name="box_inertia" params="mass x y z *origin">
+        <inertial>
+            <xacro:insert_block name="origin"/>
+            <mass value="${mass}" />
+            <inertia ixx="${(1/12) * mass * (y*y+z*z)}" ixy="0.0" ixz="0.0"
+                    iyy="${(1/12) * mass * (x*x+z*z)}" iyz="0.0"
+                    izz="${(1/12) * mass * (x*x+y*y)}" />
+        </inertial>
     </xacro:macro>
-    <xacro:macro name="box_inertia" params="m x y z">
-        <inertia ixx="${m * (y * y + z * z) / 12}" ixy="0" ixz="0" iyy="${m * (x * x + z * z) / 12}" iyz="0" izz="${m * (y * y + x * x) / 12}" />
+    <xacro:macro name="inertial_sphere" params="mass radius *origin">
+        <inertial>
+            <xacro:insert_block name="origin"/>
+            <mass value="${mass}" />
+            <inertia ixx="${(2/5) * mass * (radius*radius)}" ixy="0.0" ixz="0.0"
+                    iyy="${(2/5) * mass * (radius*radius)}" iyz="0.0"
+                    izz="${(2/5) * mass * (radius*radius)}" />
+        </inertial>
     </xacro:macro>
-    <xacro:macro name="sphere_inertia" params="m r">
-        <inertia ixx="${2 * m * r * r / 5}" ixy="0" ixz="0" iyy="${2 * m * r * r / 5}" iyz="0" izz="${2 * m * r * r / 5}" />
+    <xacro:macro name="inertial_cylinder" params="mass length radius *origin">
+        <inertial>
+            <xacro:insert_block name="origin"/>
+            <mass value="${mass}" />
+            <inertia ixx="${(1/12) * mass * (3*radius*radius + length*length)}" ixy="0.0" ixz="0.0"
+                    iyy="${(1/12) * mass * (3*radius*radius + length*length)}" iyz="0.0"
+                    izz="${(1/2) * mass * (radius*radius)}" />
+        </inertial>
     </xacro:macro>
     <!-- ............................... TROLLEY WHEEL DEFINITION .............................. -->

File: description/robot_core.xacro (robot description, xacro)
@@ -20,16 +20,36 @@
     <xacro:property name="traction_wheel_width" value="0.05"/>
     <xacro:property name="traction_track_width" value="0.6"/>
+    <xacro:property name="two_d_lidar_update_rate" value="30"/>
+    <xacro:property name="two_d_lidar_sample_size" value="361"/>
+    <xacro:property name="two_d_lidar_min_angle" value="0"/>
+    <xacro:property name="two_d_lidar_max_angle" value="360"/>
+    <xacro:property name="two_d_lidar_min_range" value="0.55"/>
+    <xacro:property name="two_d_lidar_max_range" value="16"/>
+    <xacro:property name="camera_baseline" value="0.06"/>
+    <xacro:property name="camera_height" value="0.10"/>
+    <xacro:property name="camera_horizontal_fov" value="60"/>
+    <xacro:arg name="robot_namespace" default=""/>
+    <xacro:arg name="wheel_odom_topic" default="odom" />
+    <xacro:arg name="camera_enabled" default="false" />
+    <xacro:arg name="stereo_camera_enabled" default="false" />
+    <xacro:arg name="two_d_lidar_enabled" default="false" />
+    <xacro:arg name="publish_wheel_odom_tf" default="true" />
+    <xacro:arg name="conveyor_enabled" default="false"/>
+    <xacro:arg name="ground_truth_frame" default="map"/>
+    <xacro:arg name="sim_gazebo" default="false" />
+    <xacro:arg name="sim_gz" default="false" />
+    <xacro:arg name="odometry_source" default="world" />
+    <xacro:property name="odometry_source" value="$(arg odometry_source)"/>
     <!-- LOAD MACROS -->
     <xacro:include filename="macros.xacro"/>
+    <xacro:include filename="gz.xacro"/>
     <!-- BASE LINK-->
-    <link name="base_link">
-    </link>
+    <link name="base_footprint"/>
+    <link name="base_link"/>
     <joint name="base_footprint_joint" type="fixed">
-        <parent link="base_link"/>
-        <child link="base_footprint"/>
+        <parent link="base_footprint"/>
+        <child link="base_link"/>
         <origin xyz="0 0 0" rpy="0 0 0"/>
     </joint>
-    <link name="base_footprint">
-    </link>
     <!-- CHASSIS LINK -->
     <joint name="chassis_joint" type="fixed">
@@ -54,16 +74,11 @@
             </geometry>
         </collision>
-        <inertial>
-            <mass value="${chassis_mass}" />
-            <xacro:box_inertia m="${chassis_mass}" x="${chassis_length}" y="${chassis_width}" z = "${chassis_height}"/>
-        </inertial>
-    </link>
-    <!-- MIDDLE WHEELS COLLISION AND VISUAL GEOMETRY -->
-    <!--xacro:traction_wheel cardinality="middle" dexterity="left" origin_x="0" origin_y="${traction_track_width/2}" origin_z="-${chassis_height/2+2*trolley_wheel_radius+eps-traction_wheel_radius}"/-->
-    <!--xacro:traction_wheel cardinality="middle" dexterity="right" origin_x="0" origin_y="-${traction_track_width/2}" origin_z="-${chassis_height/2+2*trolley_wheel_radius+eps-traction_wheel_radius}"/-->
+        <xacro:box_inertia mass="${chassis_mass}" x="${chassis_length}" y="${chassis_width}" z = "${chassis_height}">
+            <origin xyz="${chassis_length/2} 0 ${chassis_height/2}" rpy="0 0 0"/>
+        </xacro:box_inertia>
+    </link>
     <joint name="middle_wheel_left_joint" type="continuous">
         <parent link="base_link"/>
         <child link="middle_wheel_left_visual"/>
-        <!--origin xyz="0 ${traction_track_width/2} -${chassis_height/2+2*trolley_wheel_radius+eps-traction_wheel_radius}" rpy="-1.57 0 0"/-->
         <origin xyz="0 0.345 0" rpy="-${pi/2} 0 0"/>
         <axis xyz="0 0 1"/>
@@ -85,9 +100,17 @@
             </geometry>
         </collision>
+        <xacro:inertial_cylinder mass="${traction_wheel_mass}" length="${traction_wheel_width}" radius="${traction_wheel_radius}">
+            <origin xyz="0 0 0" rpy="0 0 0"/>
+        </xacro:inertial_cylinder>
+        <gazebo>
+            <plugin filename="ignition-gazebo-joint-state-publisher-system" name="ignition::gazebo::systems::JointStatePublisher">
+                <topic>/joint_states</topic>
+                <joint_name>Middle_wheel_left_joint</joint_name>
+            </plugin>
+        </gazebo>
     </link>
     <joint name="middle_wheel_right_joint" type="continuous">
         <parent link="base_link"/>
         <child link="middle_wheel_right_visual"/>
-        <!--origin xyz="0 -${traction_track_width/2} -${chassis_height/2+2*trolley_wheel_radius+eps-traction_wheel_radius}" rpy="1.57 0 0"/-->
         <origin xyz="0 -0.345 0" rpy="${pi/2} 0 0"/>
         <axis xyz="0 0 -1"/>
@@ -109,4 +132,13 @@
             </geometry>
         </collision>
+        <xacro:inertial_cylinder mass="${traction_wheel_mass}" length="${traction_wheel_width}" radius="${traction_wheel_radius}">
+            <origin xyz="0 0 0" rpy="0 0 0"/>
+        </xacro:inertial_cylinder>
+        <gazebo>
+            <plugin filename="ignition-gazebo-joint-state-publisher-system" name="ignition::gazebo::systems::JointStatePublisher">
+                <topic>/joint_states</topic>
+                <joint_name>Middle_wheel_right_joint</joint_name>
+            </plugin>
+        </gazebo>
     </link>
     <!-- CASTER WHEELS -->
@@ -133,4 +165,7 @@
             </geometry>
         </collision>
+        <xacro:inertial_sphere mass="${trolley_wheel_mass}" radius="${trolley_wheel_radius}">
+            <origin xyz="0 0 0" rpy="0 0 0"/>
+        </xacro:inertial_sphere>
     </link>
     <!-- Front Right Caster Wheel -->
@@ -156,4 +191,7 @@
             </geometry>
         </collision>
+        <xacro:inertial_sphere mass="${trolley_wheel_mass}" radius="${trolley_wheel_radius}">
+            <origin xyz="0 0 0" rpy="0 0 0"/>
+        </xacro:inertial_sphere>
     </link>
         <!-- back Left Caster Wheel -->
@@ -179,4 +217,7 @@
             </geometry>
         </collision>
+        <xacro:inertial_sphere mass="${trolley_wheel_mass}" radius="${trolley_wheel_radius}">
+            <origin xyz="0 0 0" rpy="0 0 0"/>
+        </xacro:inertial_sphere>
     </link>
     <!-- back Right Caster Wheel -->
@@ -202,4 +243,41 @@
             </geometry>
         </collision>
-    </link>
+        <xacro:inertial_sphere mass="${trolley_wheel_mass}" radius="${trolley_wheel_radius}">
+            <origin xyz="0 0 0" rpy="0 0 0"/>
+        </xacro:inertial_sphere>
+    </link>
+    <link name="two_d_lidar">
+            <collision>
+                <origin xyz="0 0 0" rpy="0 0 0" />
+                <geometry>
+                    <cylinder length="0.06" radius="0.075"/>
+                </geometry>
+            </collision>
+            <visual>
+                <origin xyz="0 0 0" rpy="0 0 0" />
+                <geometry>
+                    <cylinder length="0.06" radius="0.075"/>
+                </geometry>
+             <material name="black">
+                <color rgba="0.0 0.0 0.0 1.0"/>
+            </material>
+            </visual>
+            <xacro:inertial_cylinder mass="0.1" length="0.06" radius="0.075">
+                <origin xyz="0 0 0" rpy="0 0 0" />
+            </xacro:inertial_cylinder>
+    </link>
+    <joint name="two_d_lidar_joint" type="fixed">
+            <parent link="base_link"/>
+            <child link="two_d_lidar"/>
+            <origin xyz="0.0 0 0.08" rpy="0 0 0" />
+    </joint>
+        <gazebo reference="two_d_lidar">
+            <material>Gazebo/White</material>
+        </gazebo>
+    <link name="imu_frame"/>
+    <joint name="imu_joint" type="fixed">
+        <parent link="base_link"/>
+        <child link="imu_frame"/>
+        <origin xyz="0.0 0.0 0.08" rpy="0.0 0.0 0.0"/>
+    </joint>
 </robot>
