Commit message: DRIVE THE ROBOT INGINTION GAZEBO

File: description/gz.xacro (robot description, xacro)
@@ -11,5 +11,5 @@
         </plugin>
         <!-- ........................... DIFFERENTIAL DRIVE PLUGIN ................................... -->
-        <plugin filename="gz-sim-diff-drive-system" name="gz::sim::systems::DiffDrive">
+        <plugin filename="ignition-gazebo-diff-drive-system" name="ignition::gazebo::systems::DiffDrive">
             <left_joint>middle_wheel_left_joint</left_joint>
             <right_joint>middle_wheel_right_joint</right_joint>
@@ -72,6 +72,5 @@
         </gazebo>
     </xacro:if>
-    <!-- ........................... CAMERA config ................................... -->
-    <!-- ........................... IMU config ................................... -->
+     <!-- ........................... IMU config ................................... -->
     <gazebo reference="imu_frame">
         <sensor name="imu_sensor" type="imu">
@@ -83,4 +82,3 @@
         </sensor>
     </gazebo>
-    <!-- ........................... Stereo camera ................................... -->
 </robot>

File: description/macros.xacro (robot description, xacro)
@@ -38,8 +38,17 @@
                 </geometry>
             </collision>
+            <visual>
+                <origin xyz="0 0 0" rpy="0 0 0"/>
+                <geometry>
+                    <sphere radius="${trolley_wheel_radius}"/>
+                </geometry>
+                <material name="black">
+                    <color rgba="0.0 0.0 0.0 1.0"/>
+                </material>
+            </visual>
             <inertial>
                 <origin xyz="0 0 0" rpy="0 0 0" />
                 <mass value="${trolley_wheel_mass}"/>
-                <xacro:sphere_inertia m="${trolley_wheel_mass}" r="${trolley_wheel_radius}"/>
+                <xacro:inertial_sphere mass="${trolley_wheel_mass}" radius="${trolley_wheel_radius}"/>
             </inertial>
             <mu>0.0</mu>
@@ -64,8 +73,17 @@
                 <self_collide>false</self_collide>
             </collision>
+             <visual>
+                <origin xyz="0 0 0" rpy="0 0 0"/>
+                <geometry>
+                    <cylinder radius="${traction_wheel_radius}" length="${traction_wheel_width}"/>
+                </geometry>
+                <material name="plastic">
+                    <color rgba="0.1 0.1 0.1 1"/>
+                </material>
+            </visual>
             <inertial>
                 <origin xyz="0 0 0" rpy="0 ${pi/2} ${pi/2}" />
                 <mass value="${traction_wheel_mass}"/>
-                <xacro:cylinder_inertia m="${traction_wheel_mass}" r="${traction_wheel_radius}" h="${traction_wheel_width}"/>
+                <xacro:inertial_cylinder mass="${traction_wheel_mass}" radius="${traction_wheel_radius}" length="${traction_wheel_width}"/>
             </inertial>
             <mu>5.0</mu>

File: description/robot_core.xacro (robot description, xacro)
@@ -81,13 +81,14 @@
         <parent link="base_link"/>
         <child link="middle_wheel_left_visual"/>
-        <origin xyz="0 0.345 0" rpy="-${pi/2} 0 0"/>
-        <axis xyz="0 0 1"/>
+        <origin xyz="0 ${traction_track_width/2} 0" rpy="0 0 0"/>
+        <axis xyz="0 1 0" rpy="0 0 0" />
     </joint>
     <link name="middle_wheel_left_visual">
         <visual>
-            <origin xyz="0 0 0" rpy="0 0 0"/>
+             <origin xyz="0 0 0" rpy="0 ${pi/2} ${pi/2}" />
             <geometry>
                 <cylinder radius="${traction_wheel_radius}" length="${traction_wheel_width}"/>
             </geometry>
+            <self_collide>false</self_collide>
             <material name="plastic">
                 <color rgba="0.1 0.1 0.1 1"/>
@@ -95,28 +96,24 @@
         </visual>
         <collision>
-            <origin xyz="0 0 0" rpy="0 0 0"/>
+             <origin xyz="0 0 0" rpy="0 ${pi/2} ${pi/2}" />
             <geometry>
                 <cylinder radius="${traction_wheel_radius}" length="${traction_wheel_width}"/>
             </geometry>
+            <self_collide>false</self_collide>
         </collision>
         <xacro:inertial_cylinder mass="${traction_wheel_mass}" length="${traction_wheel_width}" radius="${traction_wheel_radius}">
-            <origin xyz="0 0 0" rpy="0 0 0"/>
+             <origin xyz="0 0 0" rpy="0 ${pi/2} ${pi/2}" />
         </xacro:inertial_cylinder>
-        <gazebo>
-            <plugin filename="ignition-gazebo-joint-state-publisher-system" name="ignition::gazebo::systems::JointStatePublisher">
-                <topic>/joint_states</topic>
-                <joint_name>Middle_wheel_left_joint</joint_name>
-            </plugin>
-        </gazebo>
+        <mu>5.0</mu>
     </link>
     <joint name="middle_wheel_right_joint" type="continuous">
         <parent link="base_link"/>
         <child link="middle_wheel_right_visual"/>
-        <origin xyz="0 -0.345 0" rpy="${pi/2} 0 0"/>
-        <axis xyz="0 0 -1"/>
+        <origin xyz="0 -${traction_track_width/2} 0" rpy="0 0 0"/>
+        <axis xyz="0 1 0" rpy="0 0 0" />
     </joint>
     <link name="middle_wheel_right_visual">
         <visual>
-            <origin xyz="0 0 0" rpy="0 0 0"/>
+             <origin xyz="0 0 0" rpy="0 ${pi/2} ${pi/2}" />
             <geometry>
                 <cylinder radius="${traction_wheel_radius}" length="${traction_wheel_width}"/>
@@ -125,14 +122,17 @@
                 <color rgba="0.1 0.1 0.1 1"/>
             </material>
-        </visual>
-        <collision>
-            <origin xyz="0 0 0" rpy="0 0 0"/>
+            <self_collide>false</self_collide>
+        </visual>
+        <collision>
+             <origin xyz="0 0 0" rpy="0 ${pi/2} ${pi/2}" />
             <geometry>
                 <cylinder radius="${traction_wheel_radius}" length="${traction_wheel_width}"/>
             </geometry>
+            <self_collide>false</self_collide>
         </collision>
         <xacro:inertial_cylinder mass="${traction_wheel_mass}" length="${traction_wheel_width}" radius="${traction_wheel_radius}">
-            <origin xyz="0 0 0" rpy="0 0 0"/>
+            <origin xyz="0 0 0" rpy="0 ${pi/2} ${pi/2}" />
         </xacro:inertial_cylinder>
+        <mu>5.0</mu>
         <gazebo>
             <plugin filename="ignition-gazebo-joint-state-publisher-system" name="ignition::gazebo::systems::JointStatePublisher">
@@ -142,4 +142,22 @@
         </gazebo>
     </link>
+    <transmission name="middle_wheel_left_trans">
+    <type>transmission_interface/SimpleTransmission</type>
+    <joint name="middle_wheel_left_joint">
+        <hardwareInterface>hardware_interface/VelocityJointInterface</hardwareInterface>
+    </joint>
+    <actuator name="middle_wheel_left_motor">
+        <mechanicalReduction>1</mechanicalReduction>
+    </actuator>
+    </transmission>
+    <transmission name="middle_wheel_right_trans">
+    <type>transmission_interface/SimpleTransmission</type>
+    <joint name="middle_wheel_right_joint">
+        <hardwareInterface>hardware_interface/VelocityJointInterface</hardwareInterface>
+    </joint>
+    <actuator name="middle_wheel_right_motor">
+        <mechanicalReduction>1</mechanicalReduction>
+    </actuator>
+    </transmission>
     <!-- CASTER WHEELS -->
     <!-- Front Left Caster Wheel -->
@@ -147,9 +165,10 @@
         <parent link="base_link"/>
         <child link="front_left_caster_visual"/>
-        <origin xyz="0.32 0.240 -0.02"/>
+        <origin xyz="${chassis_length/2} 0.240 -0.02"/>
+        <axis xyz="0 1 0" rpy="0 0 0" />
     </joint>
     <link name="front_left_caster_visual">
         <visual>
-            <origin xyz="0 0 0" rpy="0 0 0"/>
+            <origin xyz="0 0 0" rpy="0 ${pi/2} ${pi/2}"/>
             <geometry>
                 <sphere radius="${trolley_wheel_radius}"/>
@@ -160,5 +179,5 @@
         </visual>
         <collision>
-            <origin xyz="0 0 0" rpy="0 0 0"/>
+            <origin xyz="0 0 0" rpy="0 ${pi/2} ${pi/2}"/>
             <geometry>
                 <sphere radius="${trolley_wheel_radius}"/>
@@ -168,4 +187,5 @@
             <origin xyz="0 0 0" rpy="0 0 0"/>
         </xacro:inertial_sphere>
+         <mu>0.0</mu>
     </link>
     <!-- Front Right Caster Wheel -->
@@ -173,9 +193,10 @@
         <parent link="base_link"/>
         <child link="front_right_caster_visual"/>
-        <origin xyz="0.32 -0.240 -0.02"/>
+        <origin xyz="${chassis_length/2} -0.240 -0.02"/>
+        <axis xyz="0 1 0" rpy="0 0 0" />
     </joint>
     <link name="front_right_caster_visual">
         <visual>
-            <origin xyz="0 0 0" rpy="0 0 0"/>
+            <origin xyz="0 0 0" rpy="0 ${pi/2} ${pi/2}"/>
             <geometry>
                 <sphere radius="${trolley_wheel_radius}"/>
@@ -194,4 +215,5 @@
             <origin xyz="0 0 0" rpy="0 0 0"/>
         </xacro:inertial_sphere>
+        <mu>0.0</mu>
     </link>
         <!-- back Left Caster Wheel -->
@@ -199,9 +221,10 @@
         <parent link="base_link"/>
         <child link="back_left_caster_visual"/>
-        <origin xyz="-0.32 0.240 -0.02"/>
+        <origin xyz="-${chassis_length/2} 0.240 -0.02"/>
+        <axis xyz="0 1 0" rpy="0 0 0" />
     </joint>
     <link name="back_left_caster_visual">
         <visual>
-            <origin xyz="0 0 0" rpy="0 0 0"/>
+            <origin xyz="0 0 0" rpy="0 ${pi/2} ${pi/2}"/>
             <geometry>
                 <sphere radius="${trolley_wheel_radius}"/>
@@ -220,4 +243,5 @@
             <origin xyz="0 0 0" rpy="0 0 0"/>
         </xacro:inertial_sphere>
+         <mu>0.0</mu>
     </link>
     <!-- back Right Caster Wheel -->
@@ -225,9 +249,10 @@
         <parent link="base_link"/>
         <child link="back_right_caster_visual"/>
-        <origin xyz="-0.32 -0.240 -0.02"/>
+        <origin xyz="-${chassis_length/2} -0.240 -0.02"/>
+        <axis xyz="0 1 0" rpy="0 0 0" />
     </joint>
     <link name="back_right_caster_visual">
         <visual>
-            <origin xyz="0 0 0" rpy="0 0 0"/>
+            <origin xyz="0 0 0" rpy="0 ${pi/2} ${pi/2}"/>
             <geometry>
                 <sphere radius="${trolley_wheel_radius}"/>
@@ -246,4 +271,5 @@
             <origin xyz="0 0 0" rpy="0 0 0"/>
         </xacro:inertial_sphere>
+         <mu>0.0</mu>
     </link>
     <link name="two_d_lidar">
